File: wwgt2026badge/wwgt2026badge.kicad_pcb (KiCad board)
At the start: 2 copper layers, 100 x 70 mm, 19 parts, among them J1 Conn_01x08_Pin, J2 Conn_01x04_Pin, SW1 SW_PUSH, SW2 EC12PLGRSDVF, SW2 KEY_SWITCH, SW3 SW_PUSH, U2 rp2040-zero, U3 fj08k-s

Commit message: updated
Parts:
- moved J2 37.4 mm to (37.6, 34.5)
Connections:
- U2 pad 17: ROT_A -> /SDA1
- U2 pad 18: ROT_B -> /SCL1
- U2 pad 3: /SDA1 -> ROT_A
- U2 pad 4: /SCL1 -> ROT_B
Routing:
- net /SDA1: track 103.9 -> 12.3 mm
- net /SCL1: track 81.5 -> 8.94 mm, vias 2 -> 0
- net ROT_B: track 70.0 -> 92.3 mm
- net ROT_A: track 69.2 -> 87.2 mm
- net VCC: track 29.9 -> 12.4 mm, vias 0 -> 1
- net GND: track 233.1 -> 218.4 mm
